File: bose-qc35-usb-c.kicad_pcb (KiCad board)
At the start: 4 copper layers, 24 x 16 mm, 37 parts, among them J1 502426-2030, J2 2171790001, J3 51281-0598, Q1 BC846BM3T5G, U1 TPS25200

Commit message: Fix Molex USB-C connector footprint
Update part origin and use correct 3D model
Parts:
- moved J2 2.63 mm to (69.0, 63.1)
Changed lines of the file:
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@@
 		(locked yes)
 		(layer "B.Cu")
-		(at 70.557771 65.264483 35)
+		(at 69.049265 63.110113 35)
 		(descr "USB Type-C receptacle for USB 2.0 and PD, https://www.molex.com/en-us/products/part-detail/2171790001?display=pdf")
 		(tags "usb usb-c 2.0 pd")
@@
 			)
 		)
-		(property "Footprint" ""
+		(property "Footprint" "library:USB_C_Receptacle_Molex_2171790001"
 			(at 0 0 35)
 			(layer "F.Fab")
@@
 		(attr smd)
 		(fp_line
-			(start -4.7 -2.88)
-			(end 4.7 -2.88)
-			(stroke
-				(width 0.12)
-				(type solid)
-			)
-			(layer "B.SilkS")
-		)
-		(fp_line
-			(start -4.7 -1.6)
-			(end -4.7 -2.88)
-			(stroke
-				(width 0.12)
-				(type solid)
-			)
-			(layer "B.SilkS")
-		)
-		(fp_line
-			(start -4.7 2.6)
-			(end -4.7 0.5)
-			(stroke
-				(width 0.12)
-				(type solid)
-			)
-			(layer "B.SilkS")
-		)
-		(fp_line
-			(start 4.7 -1.600001)
-			(end 4.7 -2.88)
-			(stroke
-				(width 0.12)
-				(type solid)
-			)
-			(layer "B.SilkS")
-		)
-		(fp_line
-			(start 4.7 2.6)
-			(end 4.7 0.5)
-			(stroke
-				(width 0.12)
-				(type solid)
-			)
-			(layer "B.SilkS")
-		)
-		(fp_line
-			(start -5.32 -3.13)
-			(end 5.320001 -3.13)
+			(start -4.7 -0.25)
+			(end -4.7 1.03)
+			(stroke
+				(width 0.12)
+				(type solid)
+			)
+			(layer "B.SilkS")
+		)
+		(fp_line
+			(start -4.7 3.13)
+			(end -4.7 5.23)
+			(stroke
+				(width 0.12)
+				(type solid)
+			)
+			(layer "B.SilkS")
+		)
+		(fp_line
+			(start 4.699999 -0.25)
+			(end -4.7 -0.25)
+			(stroke
+				(width 0.12)
+				(type solid)
+			)
+			(layer "B.SilkS")
+		)
+		(fp_line
+			(start 4.699999 -0.25)
+			(end 4.7 1.03)
+			(stroke
+				(width 0.12)
+				(type solid)
+			)
+			(layer "B.SilkS")
+		)
+		(fp_line
+			(start 4.7 3.13)
+			(end 4.7 5.23)
+			(stroke
+				(width 0.12)
+				(type solid)
+			)
+			(layer "B.SilkS")
+		)
+		(fp_line
+			(start -5.32 -0.5)
+			(end -5.32 7.9)
 			(stroke
 				(width 0.05)
@@
 		)
 		(fp_line
-			(start -5.32 5.27)
-			(end -5.32 -3.13)
+			(start 5.32 -0.5)
+			(end -5.32 -0.5)
 			(stroke
 				(width 0.05)
@@
 		)
 		(fp_line
-			(start -5.32 5.27)
-			(end 5.32 5.27)
+			(start 5.32 -0.5)
+			(end 5.32 7.900001)
 			(stroke
 				(width 0.05)
@@
 		)
 		(fp_line
-			(start 5.32 5.27)
-			(end 5.320001 -3.13)
+			(start 5.32 7.900001)
+			(end -5.32 7.9)
 			(stroke
 				(width 0.05)
@@
 		)
 		(fp_line
-			(start -4.47 -2.63)
-			(end 4.470001 -2.63)
-			(stroke
-				(width 0.1)
-				(type solid)
-			)
-			(layer "B.Fab")
-		)
-		(fp_line
-			(start -4.47 3.87)
-			(end -4.47 -2.63)
-			(stroke
-				(width 0.1)
-				(type solid)
-			)
-			(layer "B.Fab")
-		)
-		(fp_line
-			(start -4.47 3.87)
-			(end 4.469999 3.87)
-			(stroke
-				(width 0.1)
-				(type solid)
-			)
-			(layer "B.Fab")
-		)
-		(fp_line
-			(start 4.469999 3.87)
-			(end 4.470001 -2.63)
+			(start -4.47 0)
+			(end -4.47 6.5)
+			(stroke
+				(width 0.1)
+				(type solid)
+			)
+			(layer "B.Fab")
+		)
+		(fp_line
+			(start 4.47 -2.05)
+			(end -4.47 -2.05)
+			(stroke
+				(width 0.1)
+				(type solid)
+			)
+			(layer "B.Fab")
+		)
+		(fp_line
+			(start 4.47 0)
+			(end -4.47 0)
+			(stroke
+				(width 0.1)
+				(type solid)
+			)
+			(layer "B.Fab")
+		)
+		(fp_line
+			(start 4.47 0)
+			(end 4.469999 6.5)
+			(stroke
+				(width 0.1)
+				(type solid)
+			)
+			(layer "B.Fab")
+		)
+		(fp_line
+			(start 4.469999 6.5)
+			(end -4.47 6.5)
 			(stroke
 				(width 0.1)
@@
 		)
 		(pad "A1" smd rect
-			(at -3.2 4.045 215)
+			(at -3.2 6.674999 215)
 			(size 0.6 1.15)
 			(layers "B.Cu" "B.Paste" "B.Mask")
@@
 		)
 		(pad "A4" smd rect
-			(at -2.4 4.045 215)
+			(at -2.4 6.675 215)
 			(size 0.6 1.15)
 			(layers "B.Cu" "B.Paste" "B.Mask")
@@
 		)
 		(pad "A5" smd rect
-			(at -1.25 4.045001 215)
+			(at -1.249999 6.675 215)
 			(size 0.3 1.15)
 			(layers "B.Cu" "B.Paste" "B.Mask")
@@
 		)
 		(pad "A6" smd rect
-			(at -0.25 4.045 215)
+			(at -0.25 6.675 215)
 			(size 0.3 1.15)
 			(layers "B.Cu" "B.Paste" "B.Mask")
@@
 		)
 		(pad "A7" smd rect
-			(at 0.25 4.045 215)
+			(at 0.25 6.675 215)
 			(size 0.3 1.15)
 			(layers "B.Cu" "B.Paste" "B.Mask")
@@
 		)
 		(pad "A8" smd rect
-			(at 1.25 4.045 215)
+			(at 1.25 6.675 215)
 			(size 0.3 1.15)
 			(layers "B.Cu" "B.Paste" "B.Mask")
@@
 		)
 		(pad "A9" smd rect
-			(at 2.4 4.045001 215)
+			(at 2.400001 6.675 215)
 			(size 0.6 1.15)
 			(layers "B.Cu" "B.Paste" "B.Mask")
@@
 		)
 		(pad "A12" smd rect
-			(at 3.2 4.045 215)
+			(at 3.2 6.675 215)
 			(size 0.6 1.15)
 			(layers "B.Cu" "B.Paste" "B.Mask")
@@
 		)
 		(pad "B1" smd rect
-			(at 3.2 4.045 215)
+			(at 3.2 6.675 215)
 			(size 0.6 1.15)
 			(layers "B.Cu" "B.Paste" "B.Mask")
@@
 		)
 		(pad "B4" smd rect
-			(at 2.4 4.045001 215)
+			(at 2.400001 6.675 215)
 			(size 0.6 1.15)
 			(layers "B.Cu" "B.Paste" "B.Mask")
@@
 		)
 		(pad "B5" smd rect
-			(at 1.75 4.045 215)
+			(at 1.75 6.675 215)
 			(size 0.3 1.15)
 			(layers "B.Cu" "B.Paste" "B.Mask")
@@
 		)
 		(pad "B6" smd rect
-			(at 0.75 4.045 215)
+			(at 0.75 6.675 215)
 			(size 0.3 1.15)
 			(layers "B.Cu" "B.Paste" "B.Mask")
@@
 		)
 		(pad "B7" smd rect
-			(at -0.75 4.045 215)
+			(at -0.75 6.675 215)
 			(size 0.3 1.15)
 			(layers "B.Cu" "B.Paste" "B.Mask")
@@
 		)
 		(pad "B8" smd rect
-			(at -1.75 4.045 215)
+			(at -1.75 6.675 215)
 			(size 0.3 1.15)
 			(layers "B.Cu" "B.Paste" "B.Mask")
@@
 		)
 		(pad "B9" smd rect
-			(at -2.4 4.045 215)
+			(at -2.4 6.675 215)
 			(size 0.6 1.15)
 			(layers "B.Cu" "B.Paste" "B.Mask")
@@
 		)
 		(pad "B12" smd rect
-			(at -3.2 4.045 215)
+			(at -3.2 6.674999 215)
 			(size 0.6 1.15)
 			(layers "B.Cu" "B.Paste" "B.Mask")
@@
 		)
 		(pad "S1" thru_hole oval
-			(at -4.32 -0.529999 215)
+			(at -4.320001 6.1 215)
+			(size 1 1.8)
+			(drill oval 0.6 1.4)
+			(layers "*.Cu" "*.Mask")
+			(remove_unused_layers no)
+			(net 12 "GND")
+			(pinfunction "SHIELD")
+			(pintype "passive")
+		)
+		(pad "S1" thru_hole oval
+			(at -4.319999 2.1 215)
 			(size 1 2.2)
 			(drill oval 0.6 1.8)
@@
 		)
 		(pad "S1" thru_hole oval
-			(at -4.32 3.47 215)
+			(at 4.32 2.1 215)
+			(size 1 2.2)
+			(drill oval 0.6 1.8)
+			(layers "*.Cu" "*.Mask")
+			(remove_unused_layers no)
+			(net 12 "GND")
+			(pinfunction "SHIELD")
+			(pintype "passive")
+		)
+		(pad "S1" thru_hole oval
+			(at 4.32 6.1 215)
 			(size 1 1.8)
 			(drill oval 0.6 1.4)
@@
 			(pintype "passive")
 		)
-		(pad "S1" thru_hole oval
-			(at 4.32 -0.53 215)
-			(size 1 2.2)
-			(drill oval 0.6 1.8)
-			(layers "*.Cu" "*.Mask")
-			(remove_unused_layers no)
-			(net 12 "GND")
-			(pinfunction "SHIELD")
-			(pintype "passive")
-		)
-		(pad "S1" thru_hole oval
-			(at 4.32 3.47 215)
-			(size 1 1.8)
-			(drill oval 0.6 1.4)
-			(layers "*.Cu" "*.Mask")
-			(remove_unused_layers no)
-			(net 12 "GND")
-			(pinfunction "SHIELD")
-			(pintype "passive")
-		)
-		(model "${KIPRJMOD}/custom_parts/HRO_TYPE-C-31-M-12.step"
+		(model "${KIPRJMOD}/custom_parts/2171790001.stp"
 			(offset
-				(xyz -4.475 -3.65 0)
+				(xyz 0 3.35 1.58)
 			)
 			(scale
@@
 			)
 			(rotate
-				(xyz 0 0 0)
-			)
-		)
+				(xyz -90 0 180)
+			)
+		)
