File: bose-qc35-usb-c.kicad_sch (KiCad schematic)
At the start: 37 parts, among them J1 502426-2030, J2 2171790001, J3 51281-0598, Q1 BC846BM3T5G, U1 TPS25200

Commit message: Update DNP components
Parts:
- H1, H2: now left out of the parts list
- J3: LCSC C127344 -> C18548053
- R1, R17, R18, R19, R2, R3, R4: now fitted
Changed lines of the file:
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@@
 		(in_bom yes)
 		(on_board yes)
-		(dnp yes)
+		(dnp no)
 		(property "Reference" "R1"
 			(at 100.838 129.6416 0)
@@
 		(in_bom yes)
 		(on_board yes)
-		(dnp yes)
+		(dnp no)
 		(property "Reference" "R2"
 			(at 128.778 129.6416 0)
@@
 		(in_bom yes)
 		(on_board yes)
-		(dnp yes)
+		(dnp no)
 		(property "Reference" "R3"
 			(at 156.718 129.6416 0)
@@
 		(in_bom yes)
 		(on_board yes)
-		(dnp yes)
+		(dnp no)
 		(property "Reference" "R4"
 			(at 184.658 129.6416 0)
@@
 			)
 		)
-		(property "LCSC" "C127344"
+		(property "LCSC" "C18548053"
 			(at 267.462 45.9232 0)
 			(effects
@@
 		(in_bom yes)
 		(on_board yes)
-		(dnp yes)
+		(dnp no)
 		(property "Reference" "R17"
 			(at 237.998 58.5216 0)
@@
 		(in_bom yes)
 		(on_board yes)
-		(dnp yes)
+		(dnp no)
 		(property "Reference" "R18"
 			(at 245.618 58.5216 0)
@@
 		(in_bom yes)
 		(on_board yes)
-		(dnp yes)
+		(dnp no)
 		(property "Reference" "R19"
 			(at 253.238 58.5216 0)
@@
 		(unit 1)
 		(exclude_from_sim no)
-		(in_bom yes)
+		(in_bom no)
 		(on_board yes)
 		(dnp no)
@@
 		(unit 1)
 		(exclude_from_sim no)
-		(in_bom yes)
+		(in_bom no)
 		(on_board yes)
 		(dnp no)
